Commit message: converted office into home

File: cpr_office_gazebo/urdf/office_geometry.urdf.xacro (robot description, xacro)
@@ -10,5 +10,5 @@
       <origin xyz="0 0 0" rpy="0 0 0"/>
       <geometry>
-        <mesh filename="package://cpr_office_gazebo/meshes/office.dae"/>
+        <mesh filename="package://cpr_office_gazebo/meshes/home.dae"/>
       </geometry>
     </visual>
@@ -16,5 +16,5 @@
       <origin xyz="0 0 0" rpy="0 0 0"/>
       <geometry>
-        <mesh filename="package://cpr_office_gazebo/meshes/office.dae"/>
+        <mesh filename="package://cpr_office_gazebo/meshes/home.dae"/>
       </geometry>
       <surface>
