Commit message: deleted unecessary files

File: cpr_inspection_gazebo/urdf/inspection_geometry.urdf.xacro (robot description, xacro)
@@ -10,5 +10,5 @@
       <origin xyz="0 0 0" rpy="0 0 0"/>
       <geometry>
-        <mesh filename="package://cpr_inspection_gazebo/meshes/inspection_world.dae"/>
+        <mesh filename="package://cpr_inspection_gazebo/meshes/inspection_world2.dae"/>
       </geometry>
     </visual>
@@ -16,5 +16,5 @@
       <origin xyz="0 0 0" rpy="0 0 0"/>
       <geometry>
-        <mesh filename="package://cpr_inspection_gazebo/meshes/inspection_world.dae"/>
+        <mesh filename="package://cpr_inspection_gazebo/meshes/inspection_world2.dae"/>
       </geometry>
       <surface>

Commit message: Cleanup and final world for solarfarm scenario

File: cpr_inspection_gazebo/urdf/inspection_geometry.urdf.xacro (robot description, xacro)
@@ -10,5 +10,5 @@
       <origin xyz="0 0 0" rpy="0 0 0"/>
       <geometry>
-        <mesh filename="package://cpr_inspection_gazebo/meshes/inspection_world2.dae"/>
+        <mesh filename="package://cpr_inspection_gazebo/meshes/inspection_hoping_its_final.dae"/>
       </geometry>
     </visual>
@@ -16,5 +16,5 @@
       <origin xyz="0 0 0" rpy="0 0 0"/>
       <geometry>
-        <mesh filename="package://cpr_inspection_gazebo/meshes/inspection_world2.dae"/>
+        <mesh filename="package://cpr_inspection_gazebo/meshes/inspection_hoping_its_final.dae"/>
       </geometry>
       <surface>

Commit message: Even more flattened version of world

File: cpr_inspection_gazebo/urdf/inspection_geometry.urdf.xacro (robot description, xacro)
@@ -10,5 +10,5 @@
       <origin xyz="0 0 0" rpy="0 0 0"/>
       <geometry>
-        <mesh filename="package://cpr_inspection_gazebo/meshes/inspection_hoping_its_final.dae"/>
+        <mesh filename="package://cpr_inspection_gazebo/meshes/inspection_wide_bridge_more_flattened.dae"/>
       </geometry>
     </visual>
@@ -16,5 +16,5 @@
       <origin xyz="0 0 0" rpy="0 0 0"/>
       <geometry>
-        <mesh filename="package://cpr_inspection_gazebo/meshes/inspection_hoping_its_final.dae"/>
+        <mesh filename="package://cpr_inspection_gazebo/meshes/inspection_wide_bridge_more_flattened.dae"/>
       </geometry>
       <surface>
